File: SeedFmSynth.kicad_sch (KiCad schematic)
At the start: 16 parts, among them J2 MIDI IN, SW1 Attack, SW2 Decay, SW3 Sustain, SW4 Release, U1 MCP23017_SS, U2 6N135

Commit message: Update to KiCad 9
Parts:
- gave numbers to parts that had none: 4
Connections:
- net +5V: no longer D1.1 (K), J1.5 (+12V), J1.6 (P6)
- net +12V: no longer names the net of D2.1 (K), J1.7 (12V), J1.8 (+12V)
- net -12V: no longer names the net of D3.2 (A), J1.15 (-12V), J1.16 (P16)
- new net: D1.1 (K), J1.5 (+12V), J1.6 (P6)
