File: SeedFmSynth.kicad_pcb (KiCad board)
At the start: 2 copper layers, 24 parts, among them J1 Eurorack_Power_16pin_Shrouded, J2 MIDI IN, J3 EuroAudioOutR, J4 EuroAudioOutL, SW1 Attack, SW2 Decay, SW3 Sustain, SW4 Release, U1 MCP23017_SS, U2 6N135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

Commit message: update to 9.07 on mac
Parts:
- U1: footprint Package_DIP:DIP-28_W7.62mm_Socket -> Package_SO:SSOP-28_5.3x10.2mm_P0.65mm
Connections:
- net +12V renamed Net-(D2-K)
- net -12V renamed Net-(D3-A)
- D1 pad 1: +5V -> Net-(D1-K)
- J1 pad 5: +5V -> Net-(D1-K)
- J1 pad 6: +5V -> Net-(D1-K)
- J3 pad 1: (no net) -> /Euro Audio/Euro Out R
- J3 pad 2: (no net) -> /Euro Audio/GND
- J4 pad 1: (no net) -> /Euro Audio/Euro Out L
- J4 pad 2: (no net) -> /Euro Audio/GND
